Commit message: add mapping

File: src/mpc_ros/xacro/hummingbird.xacro (robot description, xacro)
@@ -22,5 +22,5 @@
   <xacro:property name="rotor_velocity_slowdown_sim" value="10" />
   <xacro:property name="use_mesh_file" value="true" />
-  <xacro:property name="mesh_file" value="package://rotors_description/meshes/hummingbird.dae" />
+  <xacro:property name="mesh_file" value="$(find rotors_description)/meshes/hummingbird.dae" />
   <xacro:property name="mass" value="0.68" /> <!-- [kg] -->
   <xacro:property name="body_width" value="0.1" /> <!-- [m] -->
@@ -142,3 +142,12 @@
     <xacro:insert_block name="rotor_inertia" />
   </xacro:vertical_rotor>
+  <!-- Add realsense d435i -->
+  <xacro:include filename="$(find mpc_ros)/xacro/Realsense_DepthCam.xacro"/>
+   <xacro:realsense_d435i
+     sensor_name="camera"
+     parent_link="${namespace}/base_link"
+     rate="30">
+     <!-- <origin xyz="0 0 0.03" rpy="0 0 0 "/> -->
+     <origin xyz="0.17 0 -0.05" rpy="0 0 0 "/>
+  </xacro:realsense_d435i>
 </robot>
